Commit message: compliting the kuka control pkg and removing pkgs related to the openmanipulator

File: kuka_lbr_iiwa/kuka_lbr_iiwa_description_pkg/urdf/lbr_iiwa_14_r820_gazebo.xacro (robot description, xacro)
@@ -12,6 +12,6 @@
     </gazebo>
   </xacro:macro>
-    <!-- Gazebo Gripper Reference macro -->
-  <xacro:macro name="RefLinkGrip" params="ref">
+    <!-- Gazebo Gray Reference macro -->
+  <xacro:macro name="RefLinkGray" params="ref">
     <gazebo reference="${ref}">
       <kp>1000000.0</kp>
@@ -43,13 +43,15 @@
   <xacro:RefLink ref="link_7"/>
   <!-- tool0 -->
-  <xacro:RefLinkGrip ref="tool0"/>
+  <xacro:RefLinkGray ref="tool0"/>
   <!-- gripper_link -->
-  <xacro:RefLinkGrip ref="gripper_link"/>
+  <xacro:RefLinkGray ref="gripper_link"/>
   <!-- gripper_link_sub -->
-  <xacro:RefLinkGrip ref="gripper_link_sub"/>
+  <xacro:RefLinkGray ref="gripper_link_sub"/>
+  <!-- conveyor_belt -->
+  <xacro:RefLinkGray ref="conveyor_belt"/>
   <!-- ros_control plugin -->
   <gazebo>
     <plugin name="gazebo_ros_control" filename="libgazebo_ros_control.so">
-    <robotNamespace>/kuka_lbr_iiwa</robotNamespace>
+<!--    <robotNamespace>/kuka_lbr_iiwa</robotNamespace>-->
       <controlPeriod>0.001</controlPeriod>
       <robotSimType>gazebo_ros_control/DefaultRobotHWSim</robotSimType>

File: kuka_lbr_iiwa/kuka_lbr_iiwa_description_pkg/urdf/lbr_iiwa_14_r820_macro.xacro (robot description, xacro)
@@ -249,5 +249,5 @@
       <child link="link_1" />
       <axis xyz="0 0 1" />
-      <limit lower="-2.9668" upper="2.9668" effort="0" velocity="1.4834" />
+      <limit lower="-2.9668" upper="2.9668" effort="100" velocity="1.4834" />
     </joint>
     <joint name="joint_a2" type="revolute">
@@ -256,5 +256,5 @@
       <child link="link_2" />
       <axis xyz="0 1 0" />
-      <limit lower="-2.0942" upper="2.0942" effort="0" velocity="1.4834" />
+      <limit lower="-2.0942" upper="2.0942" effort="100" velocity="1.4834" />
     </joint>
     <joint name="joint_a3" type="revolute">
@@ -263,5 +263,5 @@
       <child link="link_3" />
       <axis xyz="0 0 1" />
-      <limit lower="-2.9668" upper="2.9668" effort="0" velocity="1.7452" />
+      <limit lower="-2.9668" upper="2.9668" effort="100" velocity="1.7452" />
     </joint>
     <joint name="joint_a4" type="revolute">
@@ -270,5 +270,5 @@
       <child link="link_4" />
       <axis xyz="0 -1 0" />
-      <limit lower="-2.0942" upper="2.0942" effort="0" velocity="1.3089" />
+      <limit lower="-2.0942" upper="2.0942" effort="100" velocity="1.3089" />
     </joint>
     <joint name="joint_a5" type="revolute">
@@ -277,5 +277,5 @@
       <child link="link_5" />
       <axis xyz="0 0 1" />
-      <limit lower="-2.9668" upper="2.9668" effort="0" velocity="2.2688" />
+      <limit lower="-2.9668" upper="2.9668" effort="100" velocity="2.2688" />
     </joint>
     <joint name="joint_a6" type="revolute">
@@ -284,5 +284,5 @@
       <child link="link_6" />
       <axis xyz="0 1 0" />
-      <limit lower="-2.0942" upper="2.0942" effort="0" velocity="2.356" />
+      <limit lower="-2.0942" upper="2.0942" effort="100" velocity="2.356" />
     </joint>
     <joint name="joint_a7" type="revolute">
@@ -291,5 +291,5 @@
       <child link="link_7" />
       <axis xyz="0 0 1" />
-      <limit lower="-3.0541" upper="3.0541" effort="0" velocity="2.356" />
+      <limit lower="-3.0541" upper="3.0541" effort="100" velocity="2.356" />
     </joint>
     <joint name="joint_a7-tool0" type="fixed">

File: kuka_lbr_iiwa/kuka_lbr_iiwa_description_pkg/urdf/lbr_iiwa_14_r820_transmission.xacro (robot description, xacro)
@@ -21,4 +21,5 @@
       </joint>
       <actuator name="motor${n}">
+        <hardwareInterface>hardware_interface/EffortJointInterface</hardwareInterface>
         <mechanicalReduction>1</mechanicalReduction>
       </actuator>
@@ -26,17 +27,17 @@
   </xacro:macro>
   <!-- Transmission 1 -->
-  <xacro:SimpleTransmissionPosition n="1" joint="joint_a1" />
+  <xacro:SimpleTransmissionEffort n="1" joint="joint_a1" />
   <!-- Transmission 2 -->
-  <xacro:SimpleTransmissionPosition n="2" joint="joint_a2" />
+  <xacro:SimpleTransmissionEffort n="2" joint="joint_a2" />
   <!-- Transmission 3 -->
-  <xacro:SimpleTransmissionPosition n="3" joint="joint_a3" />
+  <xacro:SimpleTransmissionEffort n="3" joint="joint_a3" />
   <!-- Transmission 4 -->
-  <xacro:SimpleTransmissionPosition n="4" joint="joint_a4" />
+  <xacro:SimpleTransmissionEffort n="4" joint="joint_a4" />
   <!-- Transmission 5 -->
-  <xacro:SimpleTransmissionPosition n="5" joint="joint_a5" />
+  <xacro:SimpleTransmissionEffort n="5" joint="joint_a5" />
   <!-- Transmission 6 -->
-  <xacro:SimpleTransmissionPosition n="6" joint="joint_a6" />
+  <xacro:SimpleTransmissionEffort n="6" joint="joint_a6" />
   <!-- Transmission 7 -->
-  <xacro:SimpleTransmissionPosition n="7" joint="joint_a7" />
+  <xacro:SimpleTransmissionEffort n="7" joint="joint_a7" />
   <!-- Transmission 8 -->
   <xacro:SimpleTransmissionEffort n="8" joint="gripper" />

Commit message: adding a pick and place pkg

File: kuka_lbr_iiwa/kuka_lbr_iiwa_description_pkg/urdf/lbr_iiwa_14_r820_gazebo.xacro (robot description, xacro)
@@ -15,10 +15,18 @@
   <xacro:macro name="RefLinkGray" params="ref">
     <gazebo reference="${ref}">
+      <mu1>10000</mu1>
+      <mu2>10000</mu2>
       <kp>1000000.0</kp>
-      <kd>100.0</kd>
-      <mu1>30.0</mu1>
-      <mu2>30.0</mu2>
-      <maxVel>1.0</maxVel>
+      <kd>100000.0</kd>
+      <slip1>0</slip1>
+      <slip2>0</slip2>
       <minDepth>0.001</minDepth>
+      <maxVel>0</maxVel>
+      <torsional>
+          <ode>
+              <coefficient>1000</coefficient>
+              <slip>0</slip>
+          </ode>
+      </torsional>
       <material>Gazebo/DarkGrey</material>
     </gazebo>
@@ -50,4 +58,8 @@
   <!-- conveyor_belt -->
   <xacro:RefLinkGray ref="conveyor_belt"/>
+  <!-- end effector link -->
+  <gazebo reference="end_effector_link">
+    <material>Gazebo/RedTransparent</material>
+  </gazebo>
   <!-- ros_control plugin -->
   <gazebo>

File: kuka_lbr_iiwa/kuka_lbr_iiwa_description_pkg/urdf/lbr_iiwa_14_r820_macro.xacro (robot description, xacro)
@@ -3,4 +3,7 @@
   <material name="grey">
     <color rgba="0.5 0.5 0.5 1.0"/>
+  </material>
+  <material name="red">
+    <color rgba="1.0 0 0 1.0"/>
   </material>
   <xacro:macro name="kuka_lbr_iiwa_14_r820" >
@@ -235,4 +238,21 @@
       </geometry>
     </collision>
+    <inertial>
+      <origin xyz="0 0 0" />
+      <mass value="1.0e-03" />
+      <inertia ixx="1.0e-03" ixy="0.0" ixz="0.0"
+               iyy="1.0e-03" iyz="0.0"
+               izz="1.0e-03" />
+    </inertial>
+  </link>
+  <!-- end effector link -->
+  <link name="end_effector_link">
+    <visual>
+      <origin xyz="0 0 0" rpy="0 0 0"/>
+      <geometry>
+        <box size="0.01 0.01 0.01" />
+      </geometry>
+      <material name="red"/>
+     </visual>
     <inertial>
       <origin xyz="0 0 0" />
@@ -305,5 +325,5 @@
     <origin xyz="0 0.017 0" rpy="0 -1.57 0"/>
     <axis xyz="0 1 0"/>
-    <limit velocity="4.8" effort="1" lower="-0.008" upper="0.019" />
+    <limit velocity="4.8" effort="100" lower="-0.008" upper="0.019" />
   </joint>
     <!--  Gripper joint sub -->
@@ -313,9 +333,22 @@
     <origin xyz="0 -0.017 0" rpy="0 -1.57 0"/>
     <axis xyz="0 -1 0"/>
-    <limit velocity="4.8" effort="1" lower="-0.008" upper="0.019" />
+    <limit velocity="4.8" effort="100" lower="-0.008" upper="0.019" />
     <mimic joint="gripper" multiplier="1"/>
   </joint>
+  <!-- end effector joint -->
+  <joint name="end_effector_joint" type="fixed">
+    <origin xyz="0.0 0.0 0.05" rpy="0 0 0"/>
+    <parent link="tool0"/>
+    <child link="end_effector_link"/>
+  </joint>
     <!-- ROS base_link to KUKA $ROBROOT coordinate system transform -->
-    <link name="world" />
+    <link name="world">
+      <collision>
+        <origin xyz="0.0 -0.0 -0.01" rpy="0 0 0"/>
+        <geometry>
+          <box size="2 2 0.01"/>
+        </geometry>
+      </collision>
+    </link>
     <joint name="base_link-world" type="fixed">
       <origin xyz="0 0 0" rpy="0 0 0"/>
